File: hardware/main.kicad_sch (KiCad schematic)
At the start: 34 parts, among them J2 Micro_SD_Card, SW1 SW_DIP_x01, SW2 SW_DIP_x01, SW3 SW_DIP_x01, SW4 SW_DIP_x01, SW5 SW_DIP_x01, SW6 SW_DIP_x01, SW7 SW_DIP_x01, U1 SN74LVC245APW, U2 SN74LVC245APW, U3 SN74LVC245APW, U4 Z084000xP

Commit message: add VDP
Parts:
- added C5: 0.1uF, symbol Device:C_Small
- added R16: 220, Resistor_THT:R_Axial_DIN0207_L6.3mm_D2.5mm_P7.62mm_Horizontal, symbol Device:R_Small
- C1, C2, C3, C4: value C_Small -> 0.1uF
- R1, R11, R12, R13, R14, R15, R7, R8, R9: value R_Small -> 10k
- R10: value R_Small -> 220
- R2: value R_Small -> 3.3k
- R3: value R_Small -> 1k
- R4: value R_Small -> 620
- R5: value R_Small -> 330
- R6: value R_Small -> 2k
Connections:
- net GND: now also C5.2
- net Z80_RES: now also C5.1, R16.1; no longer SW1.1
- new net: R16.2, SW1.1
Other:
- moved on the sheet: SW1
